File: elec/lea.kicad_sch (KiCad schematic)
At the start: 7 parts

Commit message: avancement des schémas et pcb
Parts:
- removed D?: D, symbol Device:D
- added C1: 1uF, Capacitor_THT:C_Axial_L3.8mm_D2.6mm_P7.50mm_Horizontal, symbol Device:C
- added C3: 10uF, Capacitor_THT:C_Radial_D6.3mm_H5.0mm_P2.50mm, symbol Device:C
- added D1: 1N4001, Diode_THT:D_DO-41_SOD81_P10.16mm_Horizontal, symbol Diode:1N4001
- C2: renamed from C?; value 22 uF -> 10uF; footprint (none) -> Capacitor_THT:C_Radial_D6.3mm_H5.0mm_P2.50mm
- J1: renamed from J?; footprint (none) -> Connector_JST:JST_XH_B3B-XH-A_1x03_P2.50mm_Vertical
- J2: renamed from J?; footprint (none) -> TerminalBlock_Phoenix:TerminalBlock_Phoenix_MKDS-1,5-2-5.08_1x02_P5.08mm_Horizontal
- J3: renamed from J?; footprint (none) -> Connector_JST:JST_XH_B2B-XH-A_1x02_P2.50mm_Vertical
- SW1: renamed from SW?; footprint (none) -> Button_Switch_THT:SW_E-Switch_EG1224_SPDT_Angled
- gave numbers to parts that had none: 1
Connections:
- net +9V: now also SW1.1 (A), C3.2, D1.1 (K)
- net GND: now also C1.2, C3.1, D1.2 (A)
- net VIN: now reaches A1.30 (VIN), C2.2, J1.2 (Pin_2), SW1.2 (B)
- net VIN: now also C1.1
- net PWM: now reaches A1.6 (D3), J1.3 (Pin_3)
- net JCK: now reaches A1.11 (D8), J3.2 (Pin_2)
Other:
- note added: "Alimentation protégée, stabilisée"
- note added: "Déclencheur minuterie"
- note added: "Servomoteur découplé"
- note removed: "Alimentation protégée par une diode en série"
- note removed: "Servomoteur découplé par une capacité de découplage en parallèle"
- company: (none) -> Top Aéro
- title: (none) -> Séparation LEA
- moved on the sheet: A1, C2, J1, J2, J3, SW1

Commit message: commit avant changement de branche
Connections:
- net +9V: now also SW1.3 (C); no longer SW1.1 (A)
- net GND: now also J3.2 (Pin_2); no longer J3.1 (Pin_1)
- net JCK: now also J3.1 (Pin_1); no longer J3.2 (Pin_2)
Changed lines of the file:
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@@
     (stroke (width 0) (type default) (color 0 0 0 0))
   )
-  (wire (pts (xy 203.2 100.33) (xy 204.47 100.33))
+  (wire (pts (xy 203.2 102.87) (xy 204.47 102.87))
     (stroke (width 0) (type default) (color 0 0 0 0))
   )
@@
     (stroke (width 0) (type default) (color 0 0 0 0))
   )
-  (wire (pts (xy 203.2 102.87) (xy 218.44 102.87))
+  (wire (pts (xy 203.2 100.33) (xy 218.44 100.33))
     (stroke (width 0) (type default) (color 0 0 0 0))
   )
@@
     (effects (font (size 1.27 1.27)) (justify left bottom))
   )
-  (label "JCK" (at 218.44 102.87 0)
+  (label "JCK" (at 218.44 100.33 0)
     (effects (font (size 1.27 1.27)) (justify left bottom))
   )
@@
     (pin "1")
   )
-  (symbol (lib_id "power:GND") (at 204.47 100.33 90) (unit 1)
-    (in_bom yes) (on_board yes) (fields_autoplaced)
-    (property "Reference" "#PWR06" (id 0) (at 210.82 100.33 0)
-      (effects (font (size 1.27 1.27)) hide)
-    )
-    (property "Value" "GND" (id 1) (at 208.28 100.3299 90)
-      (effects (font (size 1.27 1.27)) (justify right))
-    )
-    (property "Footprint" "" (id 2) (at 204.47 100.33 0)
-      (effects (font (size 1.27 1.27)) hide)
-    )
-    (property "Datasheet" "" (id 3) (at 204.47 100.33 0)
-      (effects (font (size 1.27 1.27)) hide)
-    )
-    (pin "1")
-  )
-  (symbol (lib_id "Switch:SW_SPDT") (at 144.78 64.77 0) (unit 1)
+  (symbol (lib_id "power:GND") (at 204.47 102.87 90) (unit 1)
+    (in_bom yes) (on_board yes) (fields_autoplaced)
+    (property "Reference" "#PWR06" (id 0) (at 210.82 102.87 0)
+      (effects (font (size 1.27 1.27)) hide)
+    )
+    (property "Value" "GND" (id 1) (at 208.28 102.8699 90)
+      (effects (font (size 1.27 1.27)) (justify right))
+    )
+    (property "Footprint" "" (id 2) (at 204.47 102.87 0)
+      (effects (font (size 1.27 1.27)) hide)
+    )
+    (property "Datasheet" "" (id 3) (at 204.47 102.87 0)
+      (effects (font (size 1.27 1.27)) hide)
+    )
+    (pin "1")
+  )
+  (symbol (lib_id "Switch:SW_SPDT") (at 144.78 64.77 0) (mirror x) (unit 1)
     (in_bom yes) (on_board yes)
-    (property "Reference" "SW1" (id 0) (at 148.59 57.15 0)
-      (effects (font (size 1.27 1.27)) (justify right))
-    )
-    (property "Value" "SW_SPDT" (id 1) (at 148.59 59.69 0)
-      (effects (font (size 1.27 1.27)) (justify right))
-    )
+    (property "Reference" "SW1" (id 0) (at 148.59 72.39 0)
+      (effects (font (size 1.27 1.27)) (justify right))
+    )
+    (property "Value" "SW_SPDT" (id 1) (at 148.59 69.85 0)
+      (effects (font (size 1.27 1.27)) (justify right))
+    )
